File: Untitled.kicad_pcb (KiCad board)
At the start: 2 copper layers, 229.4 x 163.7 mm, 74 parts, among them J1 Conn_02x13_Odd_Even, J10 USB_C_Receptacle_USB2.0_16P, J10_AD1 Conn_02x23_Odd_Even, J10_AD9268 Conn_02x23_Odd_Even, J11 Conn_02x08_Odd_Even, J12 Conn_02x08_Odd_Even, J13 Conn_02x08_Odd_Even, J14 Conn_02x13_Odd_Even, J15 Conn_02x08_Odd_Even, J16 Conn_02x08_Odd_Even, J17 Conn_02x05_Odd_Even, J18 DAC, J19 ADC, J2 Conn_02x13_Odd_Even, J20 Conn_02x08_Odd_Even, J21 Conn_02x08_Odd_Even, J22 Conn_02x08_Odd_Even, J23 Conn_02x13_Odd_Even, J3 Conn_02x13_Odd_Even, J4 Conn_02x13_Odd_Even, J5 Conn_02x13_Odd_Even, J6 Conn_01x04, J8 Conn_02x08_Odd_Even, U1 SN74LVC16373ADGGR, U2 SN74LVC16373ADGGR

Commit message: Update
Parts:
- removed the C1 at (68.0, 70.7)
- removed the C1 at (262.9, 47.5)
- removed C10, C11: 100nF, Capacitor_SMD:C_0805_2012Metric
- removed the C2 at (265.9, 47.5)
- removed the C2 at (66.0, 84.4)
- removed the C3 at (269.0, 47.5)
- removed the C3 at (62.0, 84.4)
- removed the C4 at (272.0, 47.5)
- removed the C4 at (61.8, 71.1)
- removed H1 (x2), H2 (x2): MountingHole, MountingHole:MountingHole_3.5mm_Pad_Via
- removed J10_AD1: Conn_02x23_Odd_Even, Connector_PinSocket_2.54mm:PinSocket_2x23_P2.54mm_Vertical
- removed J10_AD9268: Conn_02x23_Odd_Even, Connector_PinHeader_2.54mm:PinHeader_2x23_P2.54mm_Vertical
- removed J20, J21, J22, J8: Conn_02x08_Odd_Even, Connector_PinSocket_2.54mm:PinSocket_2x08_P2.54mm_Vertical
- removed J23: Conn_02x13_Odd_Even, Connector_PinHeader_2.54mm:PinHeader_2x13_P2.54mm_Vertical
- removed JP5: Jumper_2_Open, Jumper:SolderJumper-3_P1.3mm_Open_Pad1.0x1.5mm
- removed RN1, RN2, RN3, RN4: R_Pack04, Resistor_SMD:R_Array_Convex_4x0603
- removed the U1 at (40.3, 77.5)
- removed the U1 at (254.4, 44.5)
- added C1: 100nF, Capacitor_SMD:C_0805_2012Metric, F.Cu at (127.8, 37.8)
- added C12: 100nF, Capacitor_SMD:C_0805_2012Metric, B.Cu at (114.0, 85.1)
- added C13: 100nF, Capacitor_SMD:C_0805_2012Metric, B.Cu at (116.1, 75.7)
- added C14: 100nF, Capacitor_SMD:C_0805_2012Metric, B.Cu at (117.9, 79.9)
- added C15: 100nF, Capacitor_SMD:C_0805_2012Metric, B.Cu at (105.8, 76.5)
- added C16: 100nF, Capacitor_SMD:C_0805_2012Metric, B.Cu at (90.9, 81.3)
- added C17: 100nF, Capacitor_SMD:C_0805_2012Metric, B.Cu at (135.7, 83.9)
- added C18: 100nF, Capacitor_SMD:C_0805_2012Metric, B.Cu at (104.7, 82.5)
- added C19: 100nF, Capacitor_SMD:C_0805_2012Metric, B.Cu at (96.4, 73.7)
- added C2: 100nF, Capacitor_SMD:C_0805_2012Metric, F.Cu at (127.7, 39.8)
- added C20: C_Small, Capacitor_SMD:C_0805_2012Metric, B.Cu at (92.8, 66.3)
- added C21: C_Small, Capacitor_SMD:C_0805_2012Metric, B.Cu at (85.5, 66.3)
- added C22: C_Small, Capacitor_SMD:C_0805_2012Metric, B.Cu at (90.9, 77.7)
- added C23: C_Small, Capacitor_SMD:C_0805_2012Metric, B.Cu at (102.2, 81.0)
- added C24: 100nF, Capacitor_SMD:C_0805_2012Metric, B.Cu at (110.7, 71.6)
- added C25: 100nF, Capacitor_SMD:C_0805_2012Metric, B.Cu at (106.3, 84.0)
- added C26: 100nF, Capacitor_SMD:C_0805_2012Metric, F.Cu at (141.6, 87.8)
- added C3: 100nF, Capacitor_SMD:C_0805_2012Metric, F.Cu at (140.9, 40.8)
- added C4: 100nF, Capacitor_SMD:C_0805_2012Metric, F.Cu at (140.9, 38.6)
- added D1: LED, LED_SMD:LED_0805_2012Metric, F.Cu at (120.2, 62.0)
- added D2: LED, LED_SMD:LED_0805_2012Metric, F.Cu at (120.2, 59.7)
- added J10_AD2: Conn_02x23_Odd_Even, Connector_PinSocket_2.54mm:PinSocket_2x23_P2.54mm_Vertical, B.Cu at (141.0, 91.4)
- added J24: Conn_02x08_Odd_Even, Connector_PinSocket_2.54mm:PinSocket_2x08_P2.54mm_Vertical, B.Cu at (87.4, 59.4)
- added J25: Conn_02x08_Odd_Even, Connector_PinSocket_2.54mm:PinSocket_2x08_P2.54mm_Vertical, B.Cu at (100.8, 59.4)
- added J26: Conn_02x08_Odd_Even, Connector_PinSocket_2.54mm:PinSocket_2x08_P2.54mm_Vertical, B.Cu at (114.3, 59.4)
- added J27: Conn_02x13_Odd_Even, Connector_PinHeader_2.54mm:PinHeader_2x13_P2.54mm_Vertical, F.Cu at (91.9, 37.6)
- added JP6: Jumper_2_Open, Jumper:SolderJumper-3_P1.3mm_Open_Pad1.0x1.5mm, F.Cu at (115.2, 43.6)
- added JP7: Jumper_2_Open, Jumper:SolderJumper-3_P1.3mm_Open_Pad1.0x1.5mm, F.Cu at (119.0, 45.9)
- added JTAG1: CONN_02X05, Connector_PinHeader_2.54mm:PinHeader_2x05_P2.54mm_Vertical, F.Cu at (87.6, 87.6)
- added R1: 10K, Resistor_SMD:R_0603_1608Metric_Pad0.98x0.95mm_HandSolder, B.Cu at (91.4, 87.6)
- added R10: 1k, Resistor_SMD:R_0805_2012Metric, F.Cu at (151.3, 41.1)
- added R2: 10K, Resistor_SMD:R_0603_1608Metric_Pad0.98x0.95mm_HandSolder, B.Cu at (91.4, 85.1)
- added R3: 10K, Resistor_SMD:R_0603_1608Metric_Pad0.98x0.95mm_HandSolder, B.Cu at (94.8, 85.1)
- added R4: 10K, Resistor_SMD:R_0603_1608Metric_Pad0.98x0.95mm_HandSolder, B.Cu at (86.3, 74.7)
- added R5: R, Resistor_SMD:R_0603_1608Metric_Pad0.98x0.95mm_HandSolder, B.Cu at (136.1, 87.0)
- added R7: 1k, Resistor_SMD:R_0805_2012Metric, F.Cu at (120.1, 66.1)
- added R8: 1k, Resistor_SMD:R_0805_2012Metric, F.Cu at (118.0, 66.1)
- added R9: 1k, Resistor_SMD:R_0805_2012Metric, F.Cu at (137.8, 39.8)
- added RN5: R_Pack04, Resistor_SMD:R_Array_Convex_4x0603, F.Cu at (90.2, 66.0)
- added RN6: R_Pack04, Resistor_SMD:R_Array_Convex_4x0603, F.Cu at (97.1, 69.4)
- added RN7: R_Pack04, Resistor_SMD:R_Array_Convex_4x0603, F.Cu at (106.3, 65.1)
- added RN8: R_Pack04, Resistor_SMD:R_Array_Convex_4x0603, F.Cu at (114.3, 65.3)
- added RN9: R_Pack04, Resistor_SMD:R_Array_Convex_4x0603, F.Cu at (103.0, 62.8)
- added U1: TXS0108EPW, Package_SO:TSSOP-20_4.4x6.5mm_P0.65mm, F.Cu at (133.3, 39.5)
- added U3: AMS1117-3.3, Package_TO_SOT_SMD:SOT-223-3_TabPin2, B.Cu at (89.7, 69.8)
- added U4: EPM240T100, Package_QFP:LQFP-100_14x14mm_P0.5mm, F.Cu at (111.8, 78.7)
- added U5: AMS1117-1.8, Package_TO_SOT_SMD:SOT-223-3_TabPin2, B.Cu at (96.6, 80.0)
- added U6: AMS1117-3.3, Package_TO_SOT_SMD:SOT-223-3_TabPin2, F.Cu at (133.9, 64.9)
- added X1: SG-7050CCN, Oscillator:Oscillator_SMD_Abracon_ASV-4Pin_7.0x5.1mm, F.Cu at (136.0, 84.1)
- C6: value 100nF -> C_Small
- C9: value 100nF -> C_Small; moved to F.Cu
- J1, J3, J4, J5, J6: moved to F.Cu
- J11, J12: moved to B.Cu
- J17: value Conn_02x05_Odd_Even -> Conn_02x10_Odd_Even; footprint Connector_PinHeader_2.54mm:PinHeader_2x05_P2.54mm_Vertical -> Connector_PinHeader_2.54mm:PinHeader_2x10_P2.54mm_Vertical
- J2: footprint Connector_PinSocket_2.54mm:PinSocket_2x13_P2.54mm_Vertical -> Connector_PinHeader_2.54mm:PinHeader_2x13_P2.54mm_Vertical; moved to F.Cu
- U2: value SN74LVC16373ADGGR -> TXS0108EPW; footprint Package_SO:TSSOP-48_6.1x12.5mm_P0.5mm -> Package_SO:TSSOP-20_4.4x6.5mm_P0.65mm
- moved J5 242.5 mm to (30.4, 12.3), turned to 180 degrees
- moved J4 230.6 mm to (72.3, -21.1), turned to -90 degrees
- moved J1 214.4 mm to (41.9, 20.8), turned to 90 degrees
- moved J11 167.9 mm to (127.8, 59.5), turned to -45 degrees
- moved J12 162.4 mm to (141.2, 59.4), turned to -45 degrees
- moved J3 160.5 mm to (121.8, -21.1), turned to -90 degrees
- moved J2 142.6 mm to (91.4, 23.3), turned to 90 degrees
- moved J6 140.7 mm to (136.5, -21.7), turned to 90 degrees
- moved J17 117.1 mm to (129.1, 33.5), turned to 90 degrees
- moved C7 102.5 mm to (254.7, 53.5)
- moved C8 102.5 mm to (261.6, 45.6)
- moved H10 102.5 mm to (232.3, 95.0)
- moved H5 102.5 mm to (261.4, 90.6)
- moved H6 102.5 mm to (230.4, 90.6)
- moved H9 102.5 mm to (261.3, 95.0)
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Connections:
- C6 pad 1: +3V3 -> +5V
- J11 pad 1: unconnected-(J11-Pin_1-Pad1) -> /8bit_bus/D1_1
- J11 pad 10: unconnected-(J11-Pin_10-Pad10) -> /8bit_bus/CM_B_N3
- J11 pad 11: unconnected-(J11-Pin_11-Pad11) -> /8bit_bus/CM_C_P3
- J11 pad 12: unconnected-(J11-Pin_12-Pad12) -> /8bit_bus/CM_D_P4
- J11 pad 13: unconnected-(J11-Pin_13-Pad13) -> /8bit_bus/CM_CLK_M3
- J11 pad 14: unconnected-(J11-Pin_14-Pad14) -> /8bit_bus/CM_STB_N1
- J11 pad 15: unconnected-(J11-Pin_15-Pad15) -> /8bit_bus/CM_OE_M4
- J11 pad 16: unconnected-(J11-Pin_16-Pad16) -> GND
- J11 pad 2: unconnected-(J11-Pin_2-Pad2) -> /8bit_bus/D1_2
- J11 pad 3: unconnected-(J11-Pin_3-Pad3) -> /8bit_bus/D1_3
- J11 pad 4: unconnected-(J11-Pin_4-Pad4) -> GND
- J11 pad 5: unconnected-(J11-Pin_5-Pad5) -> /8bit_bus/D1_4
- J11 pad 6: unconnected-(J11-Pin_6-Pad6) -> /8bit_bus/D1_5
- J11 pad 7: unconnected-(J11-Pin_7-Pad7) -> /8bit_bus/D1_6
- J11 pad 8: unconnected-(J11-Pin_8-Pad8) -> /8bit_bus/CM_E_N4
- J11 pad 9: unconnected-(J11-Pin_9-Pad9) -> /8bit_bus/CM_A_N5
- J12 pad 1: unconnected-(J12-Pin_1-Pad1) -> /8bit_bus/D2_1
- J12 pad 14: unconnected-(J12-Pin_14-Pad14) -> Net-(J12-Pin_14)
- J12 pad 16: unconnected-(J12-Pin_16-Pad16) -> GND
- J12 pad 2: unconnected-(J12-Pin_2-Pad2) -> /8bit_bus/D2_2
- J12 pad 3: unconnected-(J12-Pin_3-Pad3) -> /8bit_bus/D2_3
- J12 pad 4: unconnected-(J12-Pin_4-Pad4) -> GND
- J12 pad 5: unconnected-(J12-Pin_5-Pad5) -> /8bit_bus/D2_4
- J12 pad 6: unconnected-(J12-Pin_6-Pad6) -> /8bit_bus/D2_5
- J12 pad 7: unconnected-(J12-Pin_7-Pad7) -> /8bit_bus/D2_6
- J17 pad 1: /3x16p-26p_adapter/VIN_5V -> /8bit_bus/D0
- J17 pad 10: unconnected-(J17-Pin_10-Pad10) -> +5V
- J17 pad 2: /3x16p-26p_adapter/VIN_5V -> /8bit_bus/D1
- J17 pad 3: GND -> /8bit_bus/D2
- J17 pad 4: GND -> /8bit_bus/D3
- J17 pad 5: unconnected-(J17-Pin_5-Pad5) -> /8bit_bus/D4
- J17 pad 6: unconnected-(J17-Pin_6-Pad6) -> /8bit_bus/D5
- J17 pad 7: unconnected-(J17-Pin_7-Pad7) -> GND
- J17 pad 8: unconnected-(J17-Pin_8-Pad8) -> /8bit_bus/A
- J17 pad 9: unconnected-(J17-Pin_9-Pad9) -> /8bit_bus/STB
- JP4 pad 1: /wide_bus_mux/VCC_5V -> +5V
- JP4 pad 2: /wide_bus_mux/VCC_J15 -> Net-(J12-Pin_14)
- U2 pad 1: /wide_bus_mux/D3_5 -> /8bit_bus/CM_CLK_M3
- U2 pad 10: GND -> Net-(U2-OE)
- U2 pad 11: /wide_bus_mux/BA6 -> GND
- U2 pad 12: /wide_bus_mux/BA7 -> /8bit_bus/D11
- U2 pad 13: /wide_bus_mux/BA8 -> /8bit_bus/D10
- U2 pad 14: /wide_bus_mux/BA9 -> /8bit_bus/D9
- U2 pad 15: GND -> /8bit_bus/D8
- U2 pad 16: /wide_bus_mux/BA10 -> /8bit_bus/D7
- U2 pad 17: /wide_bus_mux/BA11 -> /8bit_bus/D6
- U2 pad 18: +3V3 -> /8bit_bus/OE
- U2 pad 19: /wide_bus_mux/BA12 -> +5V
- U2 pad 2: /wide_bus_mux/BA0 -> +3V3
- U2 pad 20: /wide_bus_mux/BA13 -> /8bit_bus/CLK
- U2 pad 3: /wide_bus_mux/BA1 -> /8bit_bus/CM_OE_M4
- U2 pad 4: GND -> /8bit_bus/D2_1
- U2 pad 5: /wide_bus_mux/BA2 -> /8bit_bus/D2_2
- U2 pad 6: /wide_bus_mux/BA3 -> /8bit_bus/D2_3
- U2 pad 7: +3V3 -> /8bit_bus/D2_4
- U2 pad 8: /wide_bus_mux/BA4 -> /8bit_bus/D2_5
- U2 pad 9: /wide_bus_mux/BA5 -> /8bit_bus/D2_6
Routing:
- net GND: track 378.7 -> 731.1 mm, vias 11 -> 31
- net /cpld_mux/VCC_5V: track 0.00 -> 136.8 mm, vias 0 -> 6
- net +3V3: track 23.3 -> 141.9 mm, vias 4 -> 10
- net +5V: track 0.00 -> 97.9 mm, vias 0 -> 2
- net /cpld_mux/CM_CLK_M3: track 0.00 -> 58.6 mm, vias 0 -> 3
- net /wide_bus_mux/D2_1: track 50.4 -> 0.00 mm
- net /wide_bus_mux/D1_4: track 48.2 -> 0.00 mm
- net /wide_bus_mux/D2_2: track 48.1 -> 0.00 mm
- net /wide_bus_mux/D1_2: track 47.9 -> 0.00 mm
- net /wide_bus_mux/D1_1: track 47.2 -> 0.00 mm
- net /wide_bus_mux/BA2: track 46.8 -> 0.00 mm, vias 3 -> 0
- net /wide_bus_mux/BA3: track 46.5 -> 0.00 mm, vias 3 -> 0
- net /wide_bus_mux/D1_3: track 45.4 -> 0.00 mm
- net /wide_bus_mux/BA0: track 44.4 -> 0.00 mm, vias 2 -> 0
- net /wide_bus_mux/BA1: track 44.2 -> 0.00 mm, vias 2 -> 0
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- added copper zone on F.Cu, net +3V3
Other:
- board size 229.4 x 163.7 mm -> 243.8 x 207.1 mm
