File: Untitled.kicad_sch (KiCad schematic)
At the start: 12 parts, among them J1 Conn_02x13_Odd_Even, J10 USB_C_Receptacle_USB2.0_16P, J11 Conn_02x08_Odd_Even, J12 Conn_02x08_Odd_Even, J2 Conn_02x13_Odd_Even, J3 Conn_02x13_Odd_Even, J4 Conn_02x13_Odd_Even, J5 Conn_02x13_Odd_Even, J6 Conn_01x04, J7 Jack-DC, J8 Conn_02x08_Odd_Even, J9 Conn_02x10_Odd_Even

Commit message: Update
Parts:
- removed J11, J12, J8: Conn_02x08_Odd_Even, Connector_PinSocket_2.54mm:PinSocket_2x08_P2.54mm_Vertical, symbol Connector_Generic:Conn_02x08_Odd_Even
- J2: footprint Connector_PinSocket_2.54mm:PinSocket_2x13_P2.54mm_Vertical -> Connector_PinHeader_2.54mm:PinHeader_2x13_P2.54mm_Vertical
Other:
- removed sheet wide_bus_mux
- added sheet 8bit_bus (8bit_bus.kicad_sch)
- added sheet cpld_mux (cpld_mux.kicad_sch)
